Commit message: Fix: laser sensor simulation

File: ackermann_robot_control/description/urdf/ackermann_robot.gazebo.xacro (robot description, xacro)
@@ -1,187 +1,234 @@
 <?xml version="1.0"?>
-<robot name="ackermann_robot" xmlns:xacro="http://www.ros.org/wiki/xacro">
-<!-- Gazebo references -->
-<gazebo reference="chasis_link">
-  <mu1 value="0.0"/>
-  <mu2 value="0.0"/>
-  <kp  value="10000000.0" />
-  <kd  value="1.0" />
-  <material>Gazebo/Red</material>
-</gazebo>
-<gazebo reference="left_rear_wheel">
-  <mu1 value="2.0"/>
-  <mu2 value="2.0"/>
-  <kp  value="10000000.0" />
-  <kd  value="1.0" />
-  <fdir1 value="1 0 0"/>
-  <material>Gazebo/Black</material>
-</gazebo>
-<gazebo reference="right_rear_wheel">
-  <mu1 value="2.0"/>
-  <mu2 value="2.0"/>
-  <kp  value="10000000.0" />
-  <kd  value="1.0" />
-  <fdir1 value="1 0 0"/>
-  <material>Gazebo/Black</material>
-</gazebo>
-<gazebo reference="left_front_wheel">
-  <mu1 value="2.0"/>
-  <mu2 value="2.0"/>
-  <kp  value="10000000.0" />
-  <kd  value="1.0" />
-  <fdir1 value="0 0 1"/>
-  <material>Gazebo/Black</material>
-</gazebo>
-<gazebo reference="right_front_wheel">
-  <mu1 value="2.0"/>
-  <mu2 value="2.0"/>
-  <kp  value="10000000.0" />
-  <kd  value="1.0" />
-  <fdir1 value="0 0 1"/>
-  <material>Gazebo/Black</material>
-</gazebo>
-<gazebo reference="lidar">
-  <material>Gazebo/Black</material>
-</gazebo>
-<gazebo reference="camera">
-  <material>Gazebo/Black</material>
-</gazebo>
-<gazebo reference="real_sense">
-  <material>Gazebo/Grey</material>
-</gazebo>
-<!-- Gazebo Plugins -->
-<gazebo>
-  <plugin name="gazebo_ros_control" filename="libgazebo_ros_control.so">
-    <robotNamespace>/racebot</robotNamespace>
-    <robotParam>robot_description</robotParam>
-    <robotSimType>gazebo_ros_control/DefaultRobotHWSim</robotSimType>
-    <legacyModeNS>true</legacyModeNS>
-  </plugin>
-</gazebo>
-<!-- hokuyo -->
-  <gazebo reference="lidar">
-    <material>Gazebo/Grey</material>
-    <sensor type="ray" name="hokuyo_sensor">
-      <pose>0 0 0.0124 0 0 0</pose>
-      <visualize>false</visualize>
-      <update_rate>40</update_rate>
-      <ray>
-        <scan>
-          <horizontal>
-            <samples>1081</samples>
-            <resolution>1</resolution>
-            <min_angle>-2.3561944902</min_angle>
-            <max_angle>2.3561944902</max_angle>
-          </horizontal>
-        </scan>
-        <range>
-          <min>0.1</min>
-          <max>10.0</max>
-          <resolution>0.01</resolution>
-        </range>
-        <noise>
-          <mean>0.0</mean>
-          <stddev>0.01</stddev>
-        </noise>
-      </ray>
-      <plugin name="gazebo_ros_hokuyo_controller" filename="libgazebo_ros_laser.so">
-        <topicName>/scan</topicName>
-        <frameName>lidar</frameName>
+<!-- <robot name="ackermann_robot" xmlns:xacro="http://www.ros.org/wiki/xacro"> -->
+<robot xmlns:xacro="http://www.ros.org/wiki/xacro">
+  <xacro:macro name="ackermann_robot_gazebo" params="prefix">
+    <!-- Gazebo references -->
+    <gazebo reference="${prefix}chasis_link">
+      <mu1 value="0.0" />
+      <mu2 value="0.0" />
+      <kp value="10000000.0" />
+      <kd value="1.0" />
+      <material>Gazebo/Red</material>
+    </gazebo>
+    <gazebo reference="${prefix}left_rear_wheel">
+      <mu1 value="2.0" />
+      <mu2 value="2.0" />
+      <kp value="10000000.0" />
+      <kd value="1.0" />
+      <fdir1 value="1 0 0" />
+      <material>Gazebo/Black</material>
+    </gazebo>
+    <gazebo reference="${prefix}right_rear_wheel">
+      <mu1 value="2.0" />
+      <mu2 value="2.0" />
+      <kp value="10000000.0" />
+      <kd value="1.0" />
+      <fdir1 value="1 0 0" />
+      <material>Gazebo/Black</material>
+    </gazebo>
+    <gazebo reference="${prefix}left_front_wheel">
+      <mu1 value="2.0" />
+      <mu2 value="2.0" />
+      <kp value="10000000.0" />
+      <kd value="1.0" />
+      <fdir1 value="0 0 1" />
+      <material>Gazebo/Black</material>
+    </gazebo>
+    <gazebo reference="${prefix}right_front_wheel">
+      <mu1 value="2.0" />
+      <mu2 value="2.0" />
+      <kp value="10000000.0" />
+      <kd value="1.0" />
+      <fdir1 value="0 0 1" />
+      <material>Gazebo/Black</material>
+    </gazebo>
+    <gazebo reference="${prefix}lidar">
+      <material>Gazebo/Black</material>
+    </gazebo>
+    <gazebo reference="${prefix}camera">
+      <material>Gazebo/Black</material>
+    </gazebo>
+    <gazebo reference="${prefix}real_sense">
+      <material>Gazebo/Grey</material>
+    </gazebo>
+    <!-- Gazebo Plugins -->
+    <gazebo>
+      <plugin name="gazebo_ros_control" filename="libgazebo_ros_control.so">
+        <robotNamespace>/racebot</robotNamespace>
+        <robotParam>robot_description</robotParam>
+        <robotSimType>gazebo_ros_control/DefaultRobotHWSim</robotSimType>
+        <legacyModeNS>true</legacyModeNS>
       </plugin>
+    </gazebo>
+    <!-- hokuyo -->
+    <gazebo reference="${prefix}lidar">
+      <sensor type="gpu_ray" name="head_hokuyo_sensor">
+        <pose>0 0 0 0 0 0</pose>
+        <visualize>false</visualize>
+        <update_rate>40</update_rate>
+        <ray>
+          <scan>
+            <horizontal>
+              <samples>720</samples>
+              <resolution>1</resolution>
+              <min_angle>-1.570796</min_angle>
+              <max_angle>1.570796</max_angle>
+            </horizontal>
+          </scan>
+          <range>
+            <min>0.10</min>
+            <max>30.0</max>
+            <resolution>0.01</resolution>
+          </range>
+          <noise>
+            <type>gaussian</type>
+            <mean>0.0</mean>
+            <stddev>0.01</stddev>
+          </noise>
+        </ray>
+        <plugin name="gazebo_ros_head_hokuyo_controller" filename="libgazebo_ros_ray_sensor.so">
+          <ros>
+            <remapping>~/out:=scan</remapping>
+          </ros>
+          <output_type>sensor_msgs/LaserScan</output_type>
+          <frame_name>${prefix}lidar</frame_name>
+        </plugin>
+      </sensor>
+    </gazebo>
+    <!-- camera -->
+    <gazebo reference="${prefix}camera">
+      <material>Gazebo/Grey</material>
+      <sensor type="camera" name="camera">
+        <update_rate>30.0</update_rate>
+        <camera name="camera">
+          <horizontal_fov>1.3962634</horizontal_fov>
+          <image>
+            <width>800</width>
+            <height>800</height>
+            <format>R8G8B8</format>
+          </image>
+          <clip>
+            <near>0.02</near>
+            <far>300</far>
+          </clip>
+          <noise>
+            <type>gaussian</type>
+            <mean>0.0</mean>
+            <stddev>0.007</stddev>
+          </noise>
+        </camera>
+        <plugin name="camera_controller" filename="libgazebo_ros_camera.so">
+          <alwaysOn>true</alwaysOn>
+          <updateRate>0.0</updateRate>
+          <cameraName>rrbot/camera1</cameraName>
+          <imageTopicName>image_raw</imageTopicName>
+          <cameraInfoTopicName>camera_info</cameraInfoTopicName>
+          <frameName>camera</frameName>
+          <hackBaseline>0.07</hackBaseline>
+          <distortionK1>0.0</distortionK1>
+          <distortionK2>0.0</distortionK2>
+          <distortionK3>0.0</distortionK3>
+          <distortionT1>0.0</distortionT1>
+          <distortionT2>0.0</distortionT2>
+        </plugin>
+      </sensor>
+    </gazebo>
+    <!-- <gazebo reference="real_sense">
+  <sensor name="real_sense_camera" type="depth">
+    <update_rate>20</update_rate>
+    <camera>
+      <horizontal_fov>1.047198</horizontal_fov>
+      <image>
+        <width>640</width>
+        <height>480</height>
+        <format>R8G8B8</format>
+      </image>
+      <clip>
+        <near>0.05</near>
+        <far>3</far>
+      </clip>
+    </camera>
+    <plugin name="real_sense_controller" filename="libgazebo_ros_openni_kinect.so">
+      <baseline>0.2</baseline>
+      <alwaysOn>true</alwaysOn>
+      <updateRate>1.0</updateRate>
+      <cameraName>real_sense_ir</cameraName>
+      <imageTopicName>/real_sense/color/image_raw</imageTopicName>
+      <cameraInfoTopicName>/real_sense/color/camera_info</cameraInfoTopicName>
+      <depthImageTopicName>/real_sense/depth/image_raw</depthImageTopicName>
+      <depthImageInfoTopicName>/real_sense/depth/camera_info</depthImageInfoTopicName>
+      <pointCloudTopicName>/real_sense/depth/points</pointCloudTopicName>
+      <frameName>real_sense</frameName>
+      <pointCloudCutoff>0.5</pointCloudCutoff>
+      <pointCloudCutoffMax>3.0</pointCloudCutoffMax>
+      <distortionK1>0.00000001</distortionK1>
+      <distortionK2>0.00000001</distortionK2>
+      <distortionK3>0.00000001</distortionK3>
+      <distortionT1>0.00000001</distortionT1>
+      <distortionT2>0.00000001</distortionT2>
+      <CxPrime>0</CxPrime>
+      <Cx>0</Cx>
+      <Cy>0</Cy>
+      <focalLength>0</focalLength>
+      <hackBaseline>0</hackBaseline>
+    </plugin>
+  </sensor>
+</gazebo> -->
+    <!-- <gazebo reference="real_sense">
+    <sensor type="depth" name="real_sense">
+        <always_on>true</always_on>
+        <update_rate>20.0</update_rate>
+        <camera>
+            <horizontal_fov>${60.0*3.14/180.0}</horizontal_fov>
+            <image>
+                <format>R8G8B8</format>
+                <width>640</width>
+                <height>480</height>
+            </image>
+            <clip>
+                <near>0.05</near>
+                <far>8.0</far>
+            </clip>
+        </camera>
+        <plugin name="kinect_real_sense_controller" filename="libgazebo_ros_openni_kinect.so">
+            <cameraName>real_sense</cameraName>
+            <alwaysOn>true</alwaysOn>
+            <updateRate>10</updateRate>
+            <imageTopicName>rgb/image_raw</imageTopicName>
+            <depthImageTopicName>depth/image_raw</depthImageTopicName>
+            <pointCloudTopicName>depth/points</pointCloudTopicName>
+            <cameraInfoTopicName>rgb/camera_info</cameraInfoTopicName>
+            <depthImageCameraInfoTopicName>depth/camera_info</depthImageCameraInfoTopicName>
+            <frameName>realsense_depth</frameName>
+            <baseline>0.1</baseline>
+            <distortion_k1>0.0</distortion_k1>
+            <distortion_k2>0.0</distortion_k2>
+            <distortion_k3>0.0</distortion_k3>
+            <distortion_t1>0.0</distortion_t1>
+            <distortion_t2>0.0</distortion_t2>
+            <pointCloudCutoff>0.4</pointCloudCutoff>
+        </plugin>
     </sensor>
-  </gazebo>
-<!-- camera -->
-<gazebo reference="camera">
-  <material>Gazebo/Grey</material>
-    <sensor type="camera" name="camera">
-      <update_rate>30.0</update_rate>
-      <camera name="camera">
-        <horizontal_fov>1.3962634</horizontal_fov>
-        <image>
-          <width>800</width>
-          <height>800</height>
-          <format>R8G8B8</format>
-        </image>
-        <clip>
-          <near>0.02</near>
-          <far>300</far>
-        </clip>
-        <noise>
-          <type>gaussian</type>
-          <mean>0.0</mean>
-          <stddev>0.007</stddev>
-        </noise>
-      </camera>
-      <plugin name="camera_controller" filename="libgazebo_ros_camera.so">
-        <alwaysOn>true</alwaysOn>
-        <updateRate>0.0</updateRate>
-        <cameraName>rrbot/camera1</cameraName>
-        <imageTopicName>image_raw</imageTopicName>
-        <cameraInfoTopicName>camera_info</cameraInfoTopicName>
-        <frameName>camera</frameName>
-        <hackBaseline>0.07</hackBaseline>
-        <distortionK1>0.0</distortionK1>
-        <distortionK2>0.0</distortionK2>
-        <distortionK3>0.0</distortionK3>
-        <distortionT1>0.0</distortionT1>
-        <distortionT2>0.0</distortionT2>
-      </plugin>
-    </sensor>
-</gazebo>
-<gazebo reference="real_sense">
-      <sensor type="depth" name="real_sense">
-          <always_on>true</always_on>
-          <update_rate>20.0</update_rate>
-          <camera>
-              <horizontal_fov>${60.0*3.14/180.0}</horizontal_fov>
-              <image>
-                  <format>R8G8B8</format>
-                  <width>640</width>
-                  <height>480</height>
-              </image>
-              <clip>
-                  <near>0.05</near>
-                  <far>8.0</far>
-              </clip>
-          </camera>
-          <plugin name="kinect_real_sense_controller" filename="libgazebo_ros_openni_kinect.so">
-              <cameraName>real_sense</cameraName>
-              <alwaysOn>true</alwaysOn>
-              <updateRate>10</updateRate>
-              <imageTopicName>rgb/image_raw</imageTopicName>
-              <depthImageTopicName>depth/image_raw</depthImageTopicName>
-              <pointCloudTopicName>depth/points</pointCloudTopicName>
-              <cameraInfoTopicName>rgb/camera_info</cameraInfoTopicName>
-              <depthImageCameraInfoTopicName>depth/camera_info</depthImageCameraInfoTopicName>
-              <frameName>realsense_depth</frameName>
-              <baseline>0.1</baseline>
-              <distortion_k1>0.0</distortion_k1>
-              <distortion_k2>0.0</distortion_k2>
-              <distortion_k3>0.0</distortion_k3>
-              <distortion_t1>0.0</distortion_t1>
-              <distortion_t2>0.0</distortion_t2>
-              <pointCloudCutoff>0.4</pointCloudCutoff>
-          </plugin>
+</gazebo> -->
+    <gazebo reference="${prefix}imu">
+      <material>Gazebo/Orange</material>
+      <gravity>true</gravity>
+      <sensor name="imu_sensor" type="imu">
+        <always_on>true</always_on>
+        <update_rate>100</update_rate>
+        <visualize>true</visualize>
+        <topic>__default_topic__</topic>
+        <plugin filename="libgazebo_ros_imu_sensor.so" name="imu">
+          <topicName>imu</topicName>
+          <bodyName>imu</bodyName>
+          <updateRateHZ>100.0</updateRateHZ>
+          <gaussianNoise>0.0</gaussianNoise>
+          <xyzOffset>0 0 0</xyzOffset>
+          <rpyOffset>0 0 0</rpyOffset>
+          <frameName>${prefix}imu</frameName>
+        </plugin>
+        <pose>0 0 0 0 0 0</pose>
       </sensor>
-  </gazebo>
-<gazebo reference="imu">
-        <material>Gazebo/Orange</material>
-        <gravity>true</gravity>
-        <sensor name="imu_sensor" type="imu">
-            <always_on>true</always_on>
-            <update_rate>100</update_rate>
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
File: ackermann_robot_control/description/urdf/ackermann_robot.urdf.xacro (robot description, xacro)
@@ -4,7 +4,9 @@
   <xacro:include filename="$(find ackermann_robot_description)/urdf/ackermann_robot_description.urdf.xacro" />
   <xacro:include filename="$(find ackermann_robot_description)/urdf/ackermann_robot.materials.xacro" />
+  <xacro:include filename="$(find ackermann_robot_control)/urdf/ackermann_robot.gazebo.xacro" />
   <xacro:include filename="$(find ackermann_robot_control)/ros2_control/ackermann_robot.ros2_control.xacro" />
   <xacro:include filename="$(find ackermann_robot_control)/urdf/ackermann_robot.transmission.xacro" />
   <xacro:ackermann_robot prefix="$(arg prefix)" />
+  <xacro:ackermann_robot_gazebo prefix="$(arg prefix)" />
   <xacro:ackermann_robot_ros2_control prefix="$(arg prefix)" />
   <xacro:steering_hinge_transmission name="$(arg prefix)left_steering_hinge" />
@@ -14,4 +16,3 @@
   <xacro:wheel_transmission name="$(arg prefix)left_rear_wheel" />
   <xacro:wheel_transmission name="$(arg prefix)right_rear_wheel" />
-  <xacro:include filename="$(find ackermann_robot_control)/urdf/ackermann_robot.gazebo.xacro" />
 </robot>
